File: sch/shield/PKD_shield.brd.job.brd (EAGLE design)
At the start: 68.6 x 53.3 mm, 28 parts, among them IC1 74HCT244N, IC3 PIC12F683P, IC4 TL072P, Q1 BS170

Commit message: Updated shield sch
Parts:
- moved IC1 1.27 mm to (49.5, 35.6)
- moved R1 1.27 mm to (55.9, 21.6)
Routing:
- net GND: track 137.8 -> 0.00 mm
- net VCC: track 93.2 -> 0.00 mm
- net N$17: track 72.7 -> 0.00 mm
- net N$16: track 62.7 -> 0.00 mm
- net OCLK: track 57.9 -> 0.00 mm, vias 1 -> 0
- net PWR_LO: track 52.8 -> 0.00 mm
- net EMU_NOE: track 46.2 -> 0.00 mm, vias 1 -> 0
- net N$30: track 43.7 -> 0.00 mm, vias 1 -> 0
- net BIT_IN: track 42.7 -> 0.00 mm, vias 1 -> 0
- net NRST: track 42.7 -> 0.00 mm, vias 1 -> 0
- net R/E: track 42.0 -> 0.00 mm, vias 1 -> 0
- net VMID: track 41.8 -> 0.00 mm
- net LO_PKD_U: track 41.6 -> 0.00 mm
- net N$26: track 40.7 -> 0.00 mm
- net N$5: track 34.2 -> 0.00 mm
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