File: sch/shield/PKD_shield.sch (EAGLE design)
At the start: 35 parts, among them IC1 LM393N, IC2 TL084P, IC3 PIC12F683P, IC5 74HCT243N, Q1 BS170

Commit message: Updated shield sch
Parts:
- removed C4, C5: 33n, rcl:C-EU025-025X050
- removed IC2: TL084P, linear:TL084P
- removed IC5: 74HCT243N, 74xx-eu:74HCT243N
- removed R2, R5: 10k, rcl:R-EU_0207/10
- removed R3: 240k, rcl:R-EU_0207/10
- removed R6: 2,2k, rcl:R-EU_0207/10
- added IC4: TL072P, linear:TL072P
- IC1: value LM393N -> 74HCT244N; device linear:LM393N -> 74xx-eu:74HCT244N
Connections:
- removed net CROSS_LO: IC1A.OUT, IC3.GP5/T1CKI/OSC1/CLKIN, R2.1
- removed net N$28: IC1A.+IN, R3.2
- removed net N$35: IC1B.+IN, R5.1, R6.2
- removed net N$4: J3.5, J4.5
- removed net PWR_OE1: IC5A.GAB, J3.1, J4.1
- new net EMU_NOE: IC1B.G, J3.5, J4.5
- new net GEN_OE: IC1A.G, J3.1, J4.1
- new net N$5: IC1B.Y1, Q1.G
- net ANT_LO: no longer R3.1
- net GND: no longer C4.2, C5.2, IC1A.-IN, IC1P.V-, IC2P.V-, IC5A.GBA
- net LO_PKD: no longer IC1B.OUT, R5.2
- net LO_PKD_U: now also IC4A.OUT; no longer IC2A.OUT, R6.1
- net N$16: now also IC4B.+IN; no longer IC2B.+IN
- net N$26: now also IC4A.+IN; no longer IC2A.+IN
- net N$27: now also IC4A.-IN; no longer IC2A.-IN
- net N$30: now also IC1A.Y1, IC1A.Y2, IC1A.Y3, IC1A.Y4; no longer IC5A.B1, IC5A.B2, IC5A.B3, IC5A.B4
- net OCLK: no longer Q1.G
- net PWR_LO: now also IC1A.A1, IC1A.A2, IC1A.A3, IC1A.A4, IC1B.A1; no longer IC5A.A1, IC5A.A2, IC5A.A3, IC5A.A4
- net VCC: no longer C4.1, C5.1, IC1P.V+, IC2P.V+, R2.2
- net VMID: now also IC4B.-IN, IC4B.OUT; no longer IC1B.-IN, IC2B.-IN, IC2B.OUT
Other:
- note added: "SHIELD CON."
- moved on the sheet: ANALOG, J1, J2, J3, J4, J5, J6, POWER
