File: sch/shield/PKD_shield.sch (EAGLE design)
At the start: 30 parts, among them IC1 74HCT244N, IC3 PIC12F683P, IC4 TL072P, Q1 BS170

Commit message: Hardware version 1.0
Parts:
- removed IC4: TL072P, linear:TL072P
- removed J1, J2, J5, POWER: (no value), SmartPrj:PINHD-1X8TH
- removed J3: (no value), SmartPrj:PINHD-1X10TH
- removed J6: (no value), pinhead:PINHD-1X6
- removed R11: 33, rcl:R-EU_0207/10
- removed R12: 220, rcl:R-EU_0207/10
- added IC2: PIC12F683P, microchip:PIC12F683P
- added JP1: (no value), pinhead:PINHD-1X3
- added JP3: (no value), pinhead:PINHD-1X10
- added JP4, JP5, JP6, JP7: (no value), pinhead:PINHD-1X8
- added R2: 100k, rcl:R-EU_0207/10
- added R3: 510k, rcl:R-EU_0207/10
- C1: value 1n -> 100n
- C3: value 100p -> 1n
- C4: value 100n -> 100p
- IC1: value 74HCT244N -> TL072P; device 74xx-eu:74HCT244N -> linear:TL072P
- IC3: value PIC12F683P -> 74HCT244N; device microchip:PIC12F683P -> 74xx-eu:74HCT244N
- J4: device SmartPrj:PINHD-1X10TH -> pinhead:PINHD-1X6
- JP2: device pinhead:PINHD-1X3/90 -> pinhead:PINHD-1X10
- Q1: device adam:BS170 -> various:BS170
- R7: value 510k -> 33
- R8: value 100k -> 220
- renumbered R10 to R6, R9 to R5
Connections:
- net +9V: now also JP6.8, JP7.8; no longer J2.8, POWER.8
- net ANT_LO: now also JP1.3, R8.2; no longer JP2.3, R12.2
- net BIT_IN: now also IC2.GP4/AN3/T1G/OSC2/CLKOUT, JP2.4, JP3.4; no longer IC3.GP4/AN3/T1G/OSC2/CLKOUT, J3.4, J4.4
- net EMU_NOE: now also IC3B.G, JP2.5, JP3.5; no longer IC1B.G, J3.5, J4.5
- net GEN_OE: now also IC3A.G, JP2.1, JP3.1; no longer IC1A.G, J3.1, J4.1
- net GND: now also C1.2, C3.2, IC1P.V-, IC2.VSS, IC3P.GND, JP6.7, JP7.7, R2.1, R3.2; no longer C2.2, C4.2, IC1P.GND, IC3.VSS, IC4P.V-, J2.7, POWER.7, R4.1, R7.2
- net LO_PKD: now also JP4.2, JP5.2; no longer J1.2, J5.2
- net LO_PKD_U: now also C4.2, IC1A.OUT; no longer C3.2, IC4A.OUT
- net N$1: now also JP6.3, JP7.3; no longer J2.3, POWER.3
- net N$11: now also JP4.4, JP5.4; no longer J1.4, J5.4
- net N$12: now also JP4.5, JP5.5; no longer J1.5, J5.5
- net N$13: now also JP4.6, JP5.6; no longer J1.6, J5.6
- net N$14: now also JP4.7, JP5.7; no longer J1.7, J5.7
- net N$141: now also JP2.9, JP3.9; no longer J3.9, J4.9
- net N$142: now also JP2.10, JP3.10; no longer J3.10, J4.10
- net N$15: now also JP4.8, JP5.8; no longer J1.8, J5.8
- net N$16: now also IC1B.+IN, R2.2; no longer IC4B.+IN, R4.2
- net N$17: now also C3.1, R3.1; no longer C1.1, R7.1
- net N$18: now also J4.1; no longer J6.1
- net N$19: now also J4.2; no longer J6.2
- net N$20: now also J4.3; no longer J6.3
- net N$21: now also J4.4; no longer J6.4
- net N$22: now also J4.5; no longer J6.5
- net N$222: now also JP2.8, JP3.8; no longer J3.8, J4.8
- net N$223: now also JP6.4, JP7.4; no longer J2.4, POWER.4
- net N$23: now also J4.6; no longer J6.6
- net N$24: now also JP2.7, JP3.7; no longer J3.7, J4.7
- net N$25: now also JP6.6, JP7.6; no longer J2.6, POWER.6
- net N$26: now also C2.2, IC1A.+IN, R4.1; no longer C1.2, IC4A.+IN, R8.1
- net N$27: now also C4.1, IC1A.-IN; no longer C3.1, IC4A.-IN
- net N$29: now also JP1.1, R7.2; no longer JP2.1, R11.2
- net N$3: now also JP2.6, JP3.6; no longer J3.6, J4.6
- net N$30: now also IC3A.Y1, IC3A.Y2, IC3A.Y3, IC3A.Y4, R7.1; no longer IC1A.Y1, IC1A.Y2, IC1A.Y3, IC1A.Y4, R11.1
- net N$31: now also JP6.2, JP7.2; no longer J2.2, POWER.2
- net N$32: now also JP6.1, JP7.1; no longer J2.1, POWER.1
- net N$34: now also R8.1; no longer R12.1
- net N$5: now also IC3B.Y1; no longer IC1B.Y1
- net N$8: now also JP4.1, JP5.1; no longer J1.1, J5.1
- net NRST: now also IC2.GP3/!MCLR!/VPP, JP2.3, JP3.3; no longer IC3.GP3/!MCLR!/VPP, J3.3, J4.3
- net OCLK: now also IC2.GP1/AN1/CIN-/VREF/ICSPCLK, JP4.3, JP5.3; no longer IC3.GP1/AN1/CIN-/VREF/ICSPCLK, J1.3, J5.3
- net PWR_LO: now also IC2.GP2/AN2/T0CKI/INT/COUT/CCP1, IC3A.A1, IC3A.A2, IC3A.A3, IC3A.A4, IC3B.A1; no longer IC1A.A1, IC1A.A2, IC1A.A3, IC1A.A4, IC1B.A1, IC3.GP2/AN2/T0CKI/INT/COUT/CCP1
- net R/E: now also IC2.GP0/AN0/CIN+/ICSPDAT/ULPWU, JP2.2, JP3.2; no longer IC3.GP0/AN0/CIN+/ICSPDAT/ULPWU, J3.2, J4.2
- net VCC: now also C1.1, IC1P.V+, IC2.VDD, IC3P.VCC, JP6.5, JP7.5; no longer C4.1, IC1P.VCC, IC3.VDD, IC4P.V+, J2.5, POWER.5
- net VMID: now also IC1B.-IN, IC1B.OUT, R4.2; no longer IC4B.-IN, IC4B.OUT, R8.2
Other:
- moved on the sheet: C1, C2, C3, C4, R4, R7, R8

Commit message: New 3d model for v2.0
Parts:
- removed D2: 1N4148, diode:1N4148DO35-10
- added D3: 1N4148, diode:DIODE-MELF-MLL41
- added LCD1: LCD8X2, various:LCD8X2
- added R10: 3k3, rcl:R-EU_R1206
- added R11: 2k, rcl:R-EU_R1206
- added R12: 330, rcl:R-EU_R1206
- added R13: 620, rcl:R-EU_R1206
- added R14: 1k, rcl:R-EU_R1206
- added R9: (no value), pot:TRIM_EU-B25P
- added S1, S2, S3, S4, S5: (no value), switch-omron:10-XX
- C1, C2, C3, C4, C5, C6, C7: device rcl:C-EU025-025X050 -> rcl:C-EUC1206
- D1: device diode:1N4148DO35-10 -> diode:DIODE-MELF-MLL41
- IC1: value TL072P -> TL072D; device linear:TL072P -> linear:TL072D
- IC2: value PIC12F683P -> PIC12F683SN; device microchip:PIC12F683P -> microchip:PIC12F683SN; MPN (none) -> PIC12F683-I/SN; OC_FARNELL (none) -> 9759042; OC_NEWARK (none) -> 61K3434
- IC3: value 74HCT244N -> 74HCT244DW; device 74xx-eu:74HCT244N -> 74xx-eu:74HCT244DW
- R1, R2, R3, R4, R5, R6, R7, R8: device rcl:R-EU_0207/10 -> rcl:R-EU_R1206
Connections:
- removed net N$12: JP4.5, JP5.5
- removed net N$13: JP4.6, JP5.6
- removed net N$141: JP2.9, JP3.9
- removed net N$142: JP2.10, JP3.10
- removed net N$222: JP2.8, JP3.8
- removed net N$24: JP2.7, JP3.7
- new net +5V: LCD1.BL+, LCD1.VCC, R9.E
- new net DB4: JP2.7, JP3.7, LCD1.D4
- new net DB5: JP2.8, JP3.8, LCD1.D5
- new net DB6: JP2.9, JP3.9, LCD1.D6
- new net DB7: JP2.10, JP3.10, LCD1.D7
- new net E: JP4.5, JP5.5, LCD1.E
- new net N$10: R12.1, R13.2, S4.S, S4.S1
- new net N$2: LCD1.CONTR, R9.S
- new net N$6: R10.1, S1.S, S1.S1
- new net N$7: R10.2, R14.1, S2.S, S2.S1
- new net N$9: R13.1, R14.2, S3.S, S3.S1
- new net RS: JP4.6, JP5.6, LCD1.RS
- net ANT_LO: now also D3.A; no longer D1.A
- net GND: now also D1.A, LCD1.BL-, LCD1.D0, LCD1.D1, LCD1.D2, LCD1.D3, LCD1.GND, LCD1.R/W, R9.A, S1.P, S1.P1, S2.P, S2.P1, S3.P, S3.P1, S4.P, S4.P1, S5.P, S5.P1; no longer D2.A
- net N$17: now also D3.C; no longer D2.C
- net N$18: now also R11.1, R12.2, S5.S, S5.S1
Other:
- moved on the sheet: D1
