File: sch/shield/PKD_shield.brd (EAGLE design)
At the start: 68.6 x 53.3 mm, 30 parts, among them IC1 74HCT244N, IC3 PIC12F683P, IC4 TL072P, Q1 BS170

Commit message: Hardware version 1.0
Parts:
- removed IC4: TL072P, linear:DIL08
- removed J1, J2, J5, POWER: (no value), SmartPrj:1X08-TH
- removed J3: (no value), SmartPrj:1X10-TH
- removed J6: (no value), pinhead:1X06
- removed R11: 33, rcl:0207/10
- removed R12: 220, rcl:0207/10
- added IC2: PIC12F683P, microchip:DIL8
- added JP1: (no value), pinhead:1X03
- added JP3: (no value), pinhead:1X10
- added JP4, JP5, JP6, JP7: (no value), pinhead:1X08
- added R2: 100k, rcl:0207/10
- added R3: 510k, rcl:0207/10
- C1: value 1n -> 100n
- C3: value 100p -> 1n
- C4: value 100n -> 100p
- IC1: value 74HCT244N -> TL072P; device 74xx-eu:DIL20 -> linear:DIL08
- IC3: value PIC12F683P -> 74HCT244N; device microchip:DIL8 -> 74xx-eu:DIL20
- J4: device SmartPrj:1X10-TH -> pinhead:1X06
- JP2: device pinhead:1X03/90 -> pinhead:1X10
- Q1: device adam:TO92- -> various:TO92
- R7: value 510k -> 33
- R8: value 100k -> 220
- moved J4 50.9 mm to (57.1, 5.08), turned to 0 degrees
- moved C1 48.4 mm to (3.81, 15.2), turned to 270 degrees
- moved IC1 45.5 mm to (11.4, 8.89), turned to 0 degrees
- moved R8 42.7 mm to (13.1, 40.6), turned to 180 degrees
- moved IC3 39.4 mm to (48.3, 35.6), turned to 180 degrees
- moved R7 36.0 mm to (13.0, 32.6)
- moved JP2 32.7 mm to (30.2, 50.8), turned to 180 degrees
- moved C4 28.1 mm to (31.8, 17.8), turned to 0 degrees
- moved C3 27.4 mm to (58.4, 11.4)
- moved R4 15.5 mm to (48.3, 16.5)
- moved C2 6.35 mm to (52.1, 11.4), turned to 180 degrees
- moved Q1 1.28 mm to (7.62, 46.9)
- renumbered R10 to R6, R9 to R5
Connections:
- net +9V: now also JP6.8, JP7.8; no longer J2.8, POWER.8
- net ANT_LO: now also JP1.3, R8.2; no longer JP2.3, R12.2
- net BIT_IN: now also IC2.3, JP2.4, JP3.4; no longer IC3.3, J3.4, J4.4
- net EMU_NOE: now also IC3.19, JP2.5, JP3.5; no longer IC1.19, J3.5, J4.5
- net GEN_OE: now also IC3.1, JP2.1, JP3.1; no longer IC1.1, J3.1, J4.1
- net GND: now also C1.2, C3.2, IC1.4, IC2.8, IC3.10, JP6.7, JP7.7, R2.1, R3.2; no longer C2.2, C4.2, IC1.10, IC3.8, IC4.4, J2.7, POWER.7, R4.1, R7.2
- net LO_PKD: now also JP4.2, JP5.2; no longer J1.2, J5.2
- net LO_PKD_U: now also C4.2, IC1.1; no longer C3.2, IC4.1
- net N$1: now also JP6.3, JP7.3; no longer J2.3, POWER.3
- net N$11: now also JP4.4, JP5.4; no longer J1.4, J5.4
- net N$12: now also JP4.5, JP5.5; no longer J1.5, J5.5
- net N$13: now also JP4.6, JP5.6; no longer J1.6, J5.6
- net N$14: now also JP4.7, JP5.7; no longer J1.7, J5.7
- net N$141: now also JP2.9, JP3.9; no longer J3.9, J4.9
- net N$142: now also JP2.10, JP3.10; no longer J3.10, J4.10
- net N$15: now also JP4.8, JP5.8; no longer J1.8, J5.8
- net N$16: now also IC1.5, R2.2; no longer IC4.5, R4.2
- net N$17: now also C3.1, R3.1; no longer C1.1, R7.1
- net N$18: now also J4.1; no longer J6.1
- net N$19: now also J4.2; no longer J6.2
- net N$20: now also J4.3; no longer J6.3
- net N$21: now also J4.4; no longer J6.4
- net N$22: now also J4.5; no longer J6.5
- net N$222: now also JP2.8, JP3.8; no longer J3.8, J4.8
- net N$223: now also JP6.4, JP7.4; no longer J2.4, POWER.4
- net N$23: now also J4.6; no longer J6.6
- net N$24: now also JP2.7, JP3.7; no longer J3.7, J4.7
- net N$25: now also JP6.6, JP7.6; no longer J2.6, POWER.6
- net N$26: now also C2.2, IC1.3, R4.1; no longer C1.2, IC4.3, R8.1
- net N$27: now also C4.1, IC1.2; no longer C3.1, IC4.2
- net N$29: now also JP1.1, R7.2; no longer JP2.1, R11.2
- net N$3: now also JP2.6, JP3.6; no longer J3.6, J4.6
- net N$30: now also IC3.12, IC3.14, IC3.16, IC3.18, R7.1; no longer IC1.12, IC1.14, IC1.16, IC1.18, R11.1
- net N$31: now also JP6.2, JP7.2; no longer J2.2, POWER.2
- net N$32: now also JP6.1, JP7.1; no longer J2.1, POWER.1
- net N$34: now also R8.1; no longer R12.1
- net N$5: now also IC3.9; no longer IC1.9
- net N$8: now also JP4.1, JP5.1; no longer J1.1, J5.1
- net NRST: now also IC2.4, JP2.3, JP3.3; no longer IC3.4, J3.3, J4.3
- net OCLK: now also IC2.6, JP4.3, JP5.3; no longer IC3.6, J1.3, J5.3
- net PWR_LO: now also IC2.5, IC3.11, IC3.2, IC3.4, IC3.6, IC3.8; no longer IC1.11, IC1.2, IC1.4, IC1.6, IC1.8, IC3.5
- net R/E: now also IC2.7, JP2.2, JP3.2; no longer IC3.7, J3.2, J4.2
- net VCC: now also C1.1, IC1.8, IC2.1, IC3.20, JP6.5, JP7.5; no longer C4.1, IC1.20, IC3.1, IC4.8, J2.5, POWER.5
- net VMID: now also IC1.6, IC1.7, R4.2; no longer IC4.6, IC4.7, R8.2
Routing:
- net R/E: track 42.0 -> 63.9 mm, vias 1 -> 0
- net GND: track 178.7 -> 164.0 mm
- net N$17: track 71.4 -> 81.0 mm
- net N$26: track 40.7 -> 49.1 mm
- net N$16: track 62.7 -> 56.0 mm
- net OCLK: track 57.9 -> 51.7 mm, vias 1 -> 2
- net N$30: track 45.3 -> 41.2 mm, vias 1 -> 0
- net PWR_LO: track 54.4 -> 52.1 mm
- net BIT_IN: track 42.7 -> 41.9 mm, vias 1 -> 0
- net NRST: track 42.7 -> 41.9 mm, vias 1 -> 0
- net EMU_NOE: track 46.2 -> 45.5 mm, vias 1 -> 0
- net N$34: track 9.93 -> 10.6 mm
- net N$5: track 34.2 -> 34.9 mm
- net VCC: track 90.5 -> 91.1 mm
- net GEN_OE: vias 1 -> 0
Other:
- board text added: "fHID 1.0"

Commit message: New 3d model for v2.0
Parts:
- removed D2: 1N4148, diode:DO35-10
- added D3: 1N4148, diode:MELF-MLL41
- added LCD1: LCD8X2, various:LCD8X2
- added R10: 3k3, rcl:R1206
- added R11: 2k, rcl:R1206
- added R12: 330, rcl:R1206
- added R13: 620, rcl:R1206
- added R14: 1k, rcl:R1206
- added R9: (no value), pot:B25P
- added S1, S2, S3, S4, S5: (no value), switch-omron:B3F-10XX
- C1, C2, C3, C4, C5, C6, C7: device rcl:C025-025X050 -> rcl:C1206
- D1: device diode:DO35-10 -> diode:MELF-MLL41
- IC1: value TL072P -> TL072D; device linear:DIL08 -> linear:SO08
- IC2: value PIC12F683P -> PIC12F683SN; device microchip:DIL8 -> microchip:SO-08
- IC3: value 74HCT244N -> 74HCT244DW; device 74xx-eu:DIL20 -> 74xx-eu:SO20W
- R1, R2, R3, R4, R5, R6, R7, R8: device rcl:0207/10 -> rcl:R1206
- moved JP1 64.5 mm to (65.5, 18.0)
- moved Q1 60.1 mm to (65.3, 29.8), turned to 270 degrees
- moved D1 50.2 mm to (59.1, 19.1), turned to 180 degrees
- moved R7 49.6 mm to (58.8, 13.7), turned to 0 degrees
- moved R8 47.5 mm to (59.3, 29.8), turned to 0 degrees
- moved C6 39.5 mm to (61.1, 35.1), turned to 90 degrees
- moved R4 38.8 mm to (18.4, 41.3), turned to 180 degrees
- moved R3 35.7 mm to (12.7, 27.9), turned to 270 degrees
- moved C7 35.5 mm to (57.1, 35.1), turned to 90 degrees
- moved IC1 31.0 mm to (38.7, 23.5)
- moved IC2 23.9 mm to (29.8, 36.8)
- moved C1 22.8 mm to (12.7, 36.2)
- moved R5 19.6 mm to (17.1, 34.3)
- moved R6 19.4 mm to (21.0, 25.4)
- moved C4 15.7 mm to (21.0, 29.2)
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Connections:
- removed net N$12: JP4.5, JP5.5
- removed net N$13: JP4.6, JP5.6
- removed net N$141: JP2.9, JP3.9
- removed net N$142: JP2.10, JP3.10
- removed net N$222: JP2.8, JP3.8
- removed net N$24: JP2.7, JP3.7
- new net +5V: LCD1.K, LCD1.VDD, R9.E
- new net DB4: JP2.7, JP3.7, LCD1.DB4
- new net DB5: JP2.8, JP3.8, LCD1.DB5
- new net DB6: JP2.9, JP3.9, LCD1.DB6
- new net DB7: JP2.10, JP3.10, LCD1.DB7
- new net E: JP4.5, JP5.5, LCD1.E
- new net N$10: R12.1, R13.2, S4.1, S4.2
- new net N$2: LCD1.VO, R9.S
- new net N$6: R10.1, S1.1, S1.2
- new net N$7: R10.2, R14.1, S2.1, S2.2
- new net N$9: R13.1, R14.2, S3.1, S3.2
- new net RS: JP4.6, JP5.6, LCD1.RS
- net ANT_LO: now also D3.A; no longer D1.A
- net GND: now also D1.A, LCD1.A, LCD1.DB0, LCD1.DB1, LCD1.DB2, LCD1.DB3, LCD1.RW, LCD1.VSS, R9.A, S1.3, S1.4, S2.3, S2.4, S3.3, S3.4, S4.3, S4.4, S5.3, S5.4; no longer D2.A
- net N$17: now also D3.C; no longer D2.C
- net N$18: now also R11.1, R12.2, S5.1, S5.2
Routing:
- net +5V: track 0.00 -> 89.1 mm
- net E: track 0.00 -> 83.1 mm
- net RS: track 0.00 -> 77.7 mm
- net GND: track 164.0 -> 225.1 mm
- net N$18: track 2.54 -> 59.2 mm
- net R/E: track 63.9 -> 20.7 mm, vias 0 -> 1
- net N$16: track 56.0 -> 15.2 mm
- net N$9: track 0.00 -> 35.9 mm
- net N$7: track 0.00 -> 29.9 mm
- net DB5: track 0.00 -> 29.8 mm, vias 0 -> 2
- net N$2: track 0.00 -> 26.2 mm
- net DB4: track 0.00 -> 26.1 mm
- net N$10: track 0.00 -> 24.3 mm
- net BIT_IN: track 41.9 -> 19.3 mm, vias 0 -> 1
- net LO_PKD_U: track 41.6 -> 21.1 mm
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Other:
- board text added: "fHID 2.0"
- board text removed: "fHID 1.0"
